File: example_project/example_project.kicad_pcb (KiCad board)
At the start: 2 copper layers, 1 part

Commit message: print
Parts:
- added R2: R_0805_2012Metric, Resistor_SMD:R_0805_2012Metric, F.Cu at (72.2, 130.8)
- renumbered REF** to R1
Changed lines of the file:
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@@
 		(descr "Resistor SMD 0805 (2012 Metric), square (rectangular) end terminal, IPC-7351 nominal, (Body size source: IPC-SM-782 page 72, https://www.pcb-3d.com/wordpress/wp-content/uploads/ipc-sm-782a_amendment_1_and_2.pdf)")
 		(tags "resistor")
-		(property "Reference" "REF**"
+		(property "Reference" "R1"
 			(at 0 -1.65 0)
 			(layer "F.SilkS")
+			(effects
+				(font
+					(size 1 1)
+					(thickness 0.15)
+				)
+			)
+		)
+		(property "Value" "R_0805_2012Metric"
+			(at 0 1.65 0)
+			(layer "F.Fab")
+			(effects
+				(font
+					(size 1 1)
+					(thickness 0.15)
+				)
+			)
+		)
+		(property "Datasheet" ""
+			(at 0 0 0)
+			(layer "F.Fab")
+			(hide yes)
+			(effects
+				(font
+					(size 1.27 1.27)
+				)
+			)
+		)
+		(property "Description" ""
+			(at 0 0 0)
+			(layer "F.Fab")
+			(hide yes)
+			(effects
+				(font
+					(size 1.27 1.27)
+				)
+			)
+		)
+		(property "KiLib_Generator" "SMD_2terminal_chip_molded"
+			(at 0 0 0)
+			(layer "F.SilkS")
+			(hide yes)
+			(effects
+				(font
+					(size 1 1)
+					(thickness 0.15)
+				)
+			)
+		)
+		(attr smd)
+		(duplicate_pad_numbers_are_jumpers no)
+		(fp_line
+			(start -0.227064 -0.735)
+			(end 0.227064 -0.735)
+			(stroke
+				(width 0.12)
+				(type solid)
+			)
+			(layer "F.SilkS")
+		)
+		(fp_line
+			(start -0.227064 0.735)
+			(end 0.227064 0.735)
+			(stroke
+				(width 0.12)
+				(type solid)
+			)
+			(layer "F.SilkS")
+		)
+		(fp_rect
+			(start -1.68 -0.95)
+			(end 1.68 0.95)
+			(stroke
+				(width 0.05)
+				(type solid)
+			)
+			(fill no)
+			(layer "F.CrtYd")
+		)
+		(fp_rect
+			(start -1 -0.625)
+			(end 1 0.625)
+			(stroke
+				(width 0.1)
+				(type solid)
+			)
+			(fill no)
+			(layer "F.Fab")
+		)
+		(fp_text user "${REFERENCE}"
+			(at 0 0 0)
+			(layer "F.Fab")
+			(effects
+				(font
+					(size 0.5 0.5)
+					(thickness 0.08)
+				)
+			)
+		)
+		(pad "1" smd roundrect
+			(at -0.9125 0)
+			(size 1.025 1.4)
+			(layers "F.Cu" "F.Mask" "F.Paste")
+			(roundrect_rratio 0.243902)
+		)
+		(pad "2" smd roundrect
+			(at 0.9125 0)
+			(size 1.025 1.4)
+			(layers "F.Cu" "F.Mask" "F.Paste")
+			(roundrect_rratio 0.243902)
+		)
+		(embedded_fonts no)
+		(model "${KICAD10_3DMODEL_DIR}/Resistor_SMD.3dshapes/R_0805_2012Metric.step"
+			(offset
+				(xyz 0 0 0)
+			)
+			(scale
+				(xyz 1 1 1)
+			)
+			(rotate
+				(xyz 0 0 0)
+			)
+		)
+	)
+	(footprint "Resistor_SMD:R_0805_2012Metric"
+		(layer "F.Cu")
+		(at 72.25 130.85)
+		(descr "Resistor SMD 0805 (2012 Metric), square (rectangular) end terminal, IPC-7351 nominal, (Body size source: IPC-SM-782 page 72, https://www.pcb-3d.com/wordpress/wp-content/uploads/ipc-sm-782a_amendment_1_and_2.pdf)")
+		(tags "resistor")
+		(property "Reference" "R2"
+			(at 0 -1.65 0)
+			(layer "F.SilkS")

Commit message: get_edge_cuts
Other:
- board outline added: 77.1 x 33.4 mm
Changed lines of the file:
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@@
 		)
+	)
+	(gr_rect
+		(start 38.95 113.8)
+		(end 116.05 147.15)
+		(stroke
+			(width 0.05)
+			(type default)
+		)
+		(fill no)
+		(layer "Edge.Cuts")
 	)
 	(embedded_fonts no)

Commit message: make example more complicated
Parts:
- added U1: ESP32-C3-WROOM-02, RF_Module:ESP32-C3-WROOM-02, F.Cu at (87.4, 134.7)
- R1, R2: value R_0805_2012Metric -> R
Connections:
- R1 pad 1: (no net) -> Net-(U1-IO6)
- R1 pad 2: (no net) -> Net-(U1-IO3)
- R2 pad 1: (no net) -> Net-(U1-IO20/RXD)
- R2 pad 2: (no net) -> Net-(U1-IO21/TXD)

Commit message: make example more compl
Parts:
- added C1: C_Small, Capacitor_SMD:C_0805_2012Metric, F.Cu at (84.0, 140.0)
- added C2: C_Small, Capacitor_SMD:C_0805_2012Metric, F.Cu at (75.6, 141.1)
- added C3: C_Small, Capacitor_SMD:C_0805_2012Metric, F.Cu at (72.2, 141.0)
- added C4: C_Small, Capacitor_SMD:C_0805_2012Metric, F.Cu at (75.2, 139.0)
- added C5: C_Small, Capacitor_SMD:C_0805_2012Metric, F.Cu at (73.4, 143.0)
- added C6: C_Small, Capacitor_SMD:C_0805_2012Metric, F.Cu at (84.0, 141.9)
- added J1: NRJ3HF-1, Connector_Audio:Jack_6.35mm_Neutrik_NRJ3HF-1_Horizontal, F.Cu at (57.2, 123.7)
- added U2: TPS7A4101DGN, Package_SO:Texas_DGN0008B_VSSOP-8-1EP_3x3mm_P0.65mm_EP2x3mm_Mask1.88x1.98mm_ThermalVias, F.Cu at (78.3, 144.5)
- U1: value ESP32-C3-WROOM-02 -> STM32WBA55HEFx; footprint RF_Module:ESP32-C3-WROOM-02 -> Package_CSP:ST_WLCSP-41_2.98x2.76mm_Layout13x7_P0.4mm_Stagger
- moved R1 23.8 mm to (84.6, 131.3), turned to -90 degrees
- moved R2 17.0 mm to (83.2, 143.9)
- moved U1 9.52 mm to (79.8, 140.4)
Connections:
- R1 pad 1: Net-(U1-IO6) -> Net-(J1-PadS)
- R1 pad 2: Net-(U1-IO3) -> Net-(U1-PA13)
- R2 pad 1: Net-(U1-IO20/RXD) -> Net-(U1-PB15)
- R2 pad 2: Net-(U1-IO21/TXD) -> +5V
