File: example_project/example_project.kicad_sch (KiCad schematic)
At the start: 0 parts

Commit message: make example more complicated
Parts:
- added R1, R2: R, symbol Device:R
- added U1: ESP32-C3-WROOM-02, RF_Module:ESP32-C3-WROOM-02, symbol RF_Module:ESP32-C3-WROOM-02
Connections:
- new net: R2.1, U1.11 (IO20/RXD)
- new net: R2.2, U1.12 (IO21/TXD)
- new net: R1.2, U1.15 (IO3)
- new net: U1.19 (GND), U1.9 (GND)
- new net: R1.1, U1.5 (IO6)

Commit message: make example more compl
Parts:
- removed U1: ESP32-C3-WROOM-02, RF_Module:ESP32-C3-WROOM-02, symbol RF_Module:ESP32-C3-WROOM-02
- added C1, C2, C3, C4, C5, C6: C_Small, Capacitor_SMD:C_0805_2012Metric, symbol Device:C_Small
- added J1: NRJ3HF-1, Connector_Audio:Jack_6.35mm_Neutrik_NRJ3HF-1_Horizontal, symbol Connector_Audio:NRJ3HF-1
- added U1: STM32WBA55HEFx, Package_CSP:ST_WLCSP-41_2.98x2.76mm_Layout13x7_P0.4mm_Stagger, symbol MCU_ST_STM32WB:STM32WBA55HEFx
- added U2: TPS7A4101DGN, Package_SO:Texas_DGN0008B_VSSOP-8-1EP_3x3mm_P0.65mm_EP2x3mm_Mask1.88x1.98mm_ThermalVias, symbol Regulator_Linear:TPS7A4101DGN
- R1, R2: footprint (none) -> Resistor_SMD:R_0805_2012Metric
Connections:
- net at R2.1: now also U1.E4 (PB15), U2.5 (EN)
- net +5V: now reaches R2.2
- net +5V: now also C1.1, C6.1, U2.8 (IN)
- net at R1.2: now also U1.E8 (PA13)
- net at R1.1: now also J1.S
- new net: C6.2, U1.B11 (VDD11)
- new net: J1.R, U1.F1 (PA14)
- new net: J1.T, U1.F3 (PA15)
- new net: C1.2, U1.E12 (VDDA)
- new net: C3.2, U1.G4 (VDD)
- new net: C2.2, U1.A10 (VDD)
- new net: C4.2, U1.B5 (VDDANA)
- new net: C5.2, U1.C6 (VDDRFPA)
- new net +3V3: C2.1, C3.1, C4.1, C5.1, U2.1 (OUT)
- new net GND: J1.G, U1.A12 (VSSSMPS), U1.B9 (VSS), U1.D1 (VSSRF), U1.D13 (VSSA), U1.D3 (VSSRF), U1.D5 (VSSRF), U1.G6 (VSS), U2.4 (GND), U2.9 (GND)
- no-connect marks 0 -> 1
